Commit message: se agrego los stl pero falta todavia cambiarlos por los originales

File: src/pckg/urdf/wxxms.xacro (robot description, xacro)
@@ -60,10 +60,10 @@
 <link name="tilt_link_1">
   <inertial>
-    <origin xyz="0.019020433357334488 0.0003869267483030542 0.03746738590146777" rpy="0 0 0"/>
-    <mass value="0.13175271562285779"/>
-    <inertia ixx="2.8e-05" iyy="4.5e-05" izz="2.3e-05" ixy="-0.0" iyz="-0.0" ixz="-0.0"/>
-  </inertial>
-  <visual>
-    <origin xyz="0.019 0.040232 -0.1105" rpy="0 0 0"/>
+      <origin rpy="0 0 0" xyz="0 0 0.030974"/>
+      <mass value="0.127335" />
+      <inertia ixx="0.0003487000" iyy="0.0002050000" izz="0.0003045000" ixy="0" ixz="0" iyz="0" />
+    </inertial>
+  <visual>
+    <origin xyz="0 0 0" rpy="0 0 ${pi/2}"/>
     <geometry>
       <mesh filename="package://pckg/meshes/tilt_link_1.stl" scale="0.001 0.001 0.001"/>
@@ -72,5 +72,5 @@
   </visual>
   <collision>
-    <origin xyz="0.019 0.040232 -0.1105" rpy="0 0 0"/>
+    <origin xyz="0 0 0" rpy="0 0 ${pi/2}"/>
     <geometry>
       <mesh filename="package://pckg/meshes/tilt_link_1.stl" scale="0.001 0.001 0.001"/>
@@ -114,11 +114,10 @@
   </transmission>
 <joint name="tilt" type="revolute">
-  <origin xyz="-0.019 0.0 0.0415" rpy="0 0 0"/>
-  <parent link="pan_link_1"/>
-  <child link="tilt_link_1"/>
-  <axis xyz="1.0 -7e-05 -4e-06" xacro:if="${is_real}"/>
-  <axis xyz="-1.0 -7e-05 -4e-06" xacro:if="${not is_real}"/>
-  <limit upper="+1.570796" lower="-1.570796" effort="100" velocity="100"/>
-</joint>
+    <axis xyz="1 0 0"  rpy="0 0 0"/>
+    <limit effort="3" lower="${radians(-90)}" upper="${radians(90)}" velocity="${pi}"/>
+    <origin rpy="0 0 0" xyz="0 0 0.03865"/>
+    <parent link="pan_link_1"/>
+    <child link="tilt_link_1"/>
+  </joint>
 <transmission name="trans_tilt">
     <type>transmission_interface/SimpleTransmission</type>
@@ -131,5 +130,5 @@
   </transmission>
 <joint name="oakd_frame" type="fixed">
-  <origin xyz="0.018966 0.002525 0.052727" rpy="0 0 0"/>
+  <origin xyz="0 0 0.06" rpy="0 0 0"/>
   <parent link="tilt_link_1"/>
   <child link="oakd_1"/>
@@ -137,5 +136,5 @@
 <!-- camera depth joints and links -->
 	<joint name="${name}_color_joint" type="fixed">
-		<origin xyz="0 -0.0370 0.018" rpy="0 0 ${-pi/2}"/>
+		<origin xyz="0 0 0" rpy="0 0 ${-pi/2}"/>
 		<parent link="oakd_1"/>
 		<child link="${name}_color_frame" />

Commit message: YA FUNCIONAAAAA solo falta arreglar el pantilt posicion porque choca con lidar

File: src/pckg/urdf/wxxms.xacro (robot description, xacro)
@@ -4,4 +4,6 @@
 <xacro:include filename="$(find pckg)/urdf/materials.xacro" />
 <xacro:include filename="$(find pckg)/urdf/oakd.gazebo" />
+<xacro:include filename="$(find jackal_description)/urdf/jackal.urdf.xacro">
+</xacro:include>
     <xacro:property name="flag_color" value="1"/>
     <xacro:property name="flag_depth" value="0"/>
@@ -12,11 +14,11 @@
     <xacro:property name="real" value="$(arg is_real)" />
 <xacro:if value="$(arg use_world_frame)">
-    <link name="world"/>
+    <!--<link name="world"/>-->
     <joint name="fixed" type="fixed">
-      <parent link="world"/>
-      <child link="base_link"/>
+      <parent link="mid_mount"/>
+      <child link="base_linkT"/>
     </joint>
 </xacro:if>
-<link name="base_link">
+<link name="base_linkT">
   <inertial>
     <origin xyz="1.2967337914845635e-06 -0.008768228394477627 0.026298757012131167" rpy="0 0 0"/>
@@ -100,5 +102,5 @@
 <joint name="pan" type="continuous">
   <origin xyz="0.0 -0.040232 0.069" rpy="0 0 0"/>
-  <parent link="base_link"/>
+  <parent link="base_linkT"/>
   <child link="pan_link_1"/>
   <axis xyz="0.0 0.0 1.0"/>
